Commit message: ajout du fichier urdf

File: fichiers_physiques/robot.urdf (robot description, URDF)
Before this commit: robot onshape, 1 links, 0 joints
Links:
- added link part_11; collision mesh filename=package:///part_11.stl; visual mesh filename=package:///part_11.stl
- added link part_2; collision mesh filename=package:///part_2.stl; visual mesh filename=package:///part_2.stl
- added link part_4; collision mesh filename=package:///part_4.stl; visual mesh filename=package:///part_4.stl
- added link part_5; collision mesh filename=package:///part_5.stl; visual mesh filename=package:///part_5.stl
- added link part_6; collision mesh filename=package:///part_6.stl; visual mesh filename=package:///part_6.stl
- added link part_7; collision mesh filename=package:///part_7.stl; visual mesh filename=package:///part_7.stl
- added link poignee; collision mesh filename=package:///poignee.stl; visual mesh filename=package:///poignee.stl
- added link support_pince; collision mesh filename=package:///support_pince.stl; visual mesh filename=package:///support_pince.stl
- link part_1: geometry collision mesh filename=package:///part_1.stl; visual mesh filename=package:///part_1.stl
