Commit message: add .stl to meshes directory

File: catkin_ws/src/braccio_description/urdf/robot.urdf (robot description, URDF)
Before this commit: robot onshape, 9 links, 0 joints
Links:
- link part_1: geometry collision mesh filename=package:///meshes/part_1.stl; visual mesh filename=package:///meshes/part_1.stl
- link part_11: geometry collision mesh filename=package:///meshes/part_11.stl; visual mesh filename=package:///meshes/part_11.stl
- link part_2: geometry collision mesh filename=package:///meshes/part_2.stl; visual mesh filename=package:///meshes/part_2.stl
- link part_4: geometry collision mesh filename=package:///meshes/part_4.stl; visual mesh filename=package:///meshes/part_4.stl
- link part_5: geometry collision mesh filename=package:///meshes/part_5.stl; visual mesh filename=package:///meshes/part_5.stl
- link part_6: geometry collision mesh filename=package:///meshes/part_6.stl; visual mesh filename=package:///meshes/part_6.stl
- link part_7: geometry collision mesh filename=package:///meshes/part_7.stl; visual mesh filename=package:///meshes/part_7.stl
- link poignee: geometry collision mesh filename=package:///meshes/poignee.stl; visual mesh filename=package:///meshes/poignee.stl
- link support_pince: geometry collision mesh filename=package:///meshes/support_pince.stl; visual mesh filename=package:///meshes/support_pince.stl

Commit message: ajout du git de poopy pour avoir un modele urdf

File: catkin_ws/src/braccio_description/urdf/robot.urdf (robot description, URDF)
Before this commit: robot onshape, 9 links, 0 joints
Links:
- link part_1: geometry collision mesh filename=package://braccio_description/meshes/part_1.stl; visual mesh filename=package://braccio_description/meshes/part_1.stl
- link part_11: geometry collision mesh filename=package://braccio_description/meshes/part_11.stl; visual mesh filename=package://braccio_description/meshes/part_11.stl
- link part_2: geometry collision mesh filename=package://braccio_description/meshes/part_2.stl; visual mesh filename=package://braccio_description/meshes/part_2.stl
- link part_4: geometry collision mesh filename=package://braccio_description/meshes/part_4.stl; visual mesh filename=package://braccio_description/meshes/part_4.stl
- link part_5: geometry collision mesh filename=package://braccio_description/meshes/part_5.stl; visual mesh filename=package://braccio_description/meshes/part_5.stl
- link part_6: geometry collision mesh filename=package://braccio_description/meshes/part_6.stl; visual mesh filename=package://braccio_description/meshes/part_6.stl
- link part_7: geometry collision mesh filename=package://braccio_description/meshes/part_7.stl; visual mesh filename=package://braccio_description/meshes/part_7.stl
- link poignee: geometry collision mesh filename=package://braccio_description/meshes/poignee.stl; visual mesh filename=package://braccio_description/meshes/poignee.stl
- link support_pince: geometry collision mesh filename=package://braccio_description/meshes/support_pince.stl; visual mesh filename=package://braccio_description/meshes/support_pince.stl

Commit message: fichiers URDF du Braccio correctement générés

File: catkin_ws/src/braccio_description/urdf/robot.urdf (robot description, URDF)
Before this commit: robot onshape, 9 links, 0 joints
Links:
- added link base_link, mass 0; collision mesh filename=package://braccio_description/meshes/base_link_collision.stl; visual mesh filename=package://braccio_description/meshes/base_link_visual.stl
- added link part_11_2, mass 0; collision mesh filename=package://braccio_description/meshes/part_11_2_collision.stl; visual mesh filename=package://braccio_description/meshes/part_11_2_visual.stl
- added link part_17, mass 0; collision mesh filename=package://braccio_description/meshes/part_17_collision.stl; visual mesh filename=package://braccio_description/meshes/part_17_visual.stl
- added link part_1_10, mass 0.0598161; collision mesh filename=package://braccio_description/meshes/part_1_10_collision.stl; visual mesh filename=package://braccio_description/meshes/part_1_10_visual.stl
- added link part_1_2, mass 0; collision mesh filename=package://braccio_description/meshes/part_1_2_collision.stl; visual mesh filename=package://braccio_description/meshes/part_1_2_visual.stl
- added link part_1_3, mass 0; collision mesh filename=package://braccio_description/meshes/part_1_3_collision.stl; visual mesh filename=package://braccio_description/meshes/part_1_3_visual.stl
- added link part_1_4, mass 0; collision mesh filename=package://braccio_description/meshes/part_1_4_collision.stl; visual mesh filename=package://braccio_description/meshes/part_1_4_visual.stl
- added link part_1_5, mass 0; collision mesh filename=package://braccio_description/meshes/part_1_5_collision.stl; visual mesh filename=package://braccio_description/meshes/part_1_5_visual.stl
- added link part_1_6, mass 0; collision mesh filename=package://braccio_description/meshes/part_1_6_collision.stl; visual mesh filename=package://braccio_description/meshes/part_1_6_visual.stl
- added link part_1_7, mass 0; collision mesh filename=package://braccio_description/meshes/part_1_7_collision.stl; visual mesh filename=package://braccio_description/meshes/part_1_7_visual.stl
- added link part_1_8, mass 0; collision mesh filename=package://braccio_description/meshes/part_1_8_collision.stl; visual mesh filename=package://braccio_description/meshes/part_1_8_visual.stl
- added link part_1_9, mass 0; collision mesh filename=package://braccio_description/meshes/part_1_9_collision.stl; visual mesh filename=package://braccio_description/meshes/part_1_9_visual.stl
- added link part_2_2, mass 0; collision mesh filename=package://braccio_description/meshes/part_2_2_collision.stl; visual mesh filename=package://braccio_description/meshes/part_2_2_visual.stl
- added link part_4_2, mass 0; collision mesh filename=package://braccio_description/meshes/part_4_2_collision.stl; visual mesh filename=package://braccio_description/meshes/part_4_2_visual.stl
- added link part_5_2, mass 0; collision mesh filename=package://braccio_description/meshes/part_5_2_collision.stl; visual mesh filename=package://braccio_description/meshes/part_5_2_visual.stl
- added link part_6_2, mass 0; collision mesh filename=package://braccio_description/meshes/part_6_2_collision.stl; visual mesh filename=package://braccio_description/meshes/part_6_2_visual.stl
- added link part_6_3, mass 0; collision mesh filename=package://braccio_description/meshes/part_6_3_collision.stl; visual mesh filename=package://braccio_description/meshes/part_6_3_visual.stl
- added link part_7_2, mass 0; collision mesh filename=package://braccio_description/meshes/part_7_2_collision.stl; visual mesh filename=package://braccio_description/meshes/part_7_2_visual.stl
- link part_1: mass 0.0598161 -> 0; geometry collision mesh filename=package://braccio_description/meshes/part_1_collision.stl; visual mesh filename=package://braccio_description/meshes/part_1_visual.stl
- link part_11: mass None -> 0; geometry collision mesh filename=package://braccio_description/meshes/part_11_collision.stl; visual mesh filename=package://braccio_description/meshes/part_11_visual.stl
- link part_2: mass None -> 0; geometry collision mesh filename=package://braccio_description/meshes/part_2_collision.stl; visual mesh filename=package://braccio_description/meshes/part_2_visual.stl
- link part_4: mass None -> 0; geometry collision mesh filename=package://braccio_description/meshes/part_4_collision.stl; visual mesh filename=package://braccio_description/meshes/part_4_visual.stl
- link part_5: mass None -> 0; geometry collision mesh filename=package://braccio_description/meshes/part_5_collision.stl; visual mesh filename=package://braccio_description/meshes/part_5_visual.stl
- link part_6: mass None -> 0; geometry collision mesh filename=package://braccio_description/meshes/part_6_collision.stl; visual mesh filename=package://braccio_description/meshes/part_6_visual.stl
- link part_7: mass None -> 0; geometry collision mesh filename=package://braccio_description/meshes/part_7_collision.stl; visual mesh filename=package://braccio_description/meshes/part_7_visual.stl
- link poignee: mass None -> 0; geometry collision mesh filename=package://braccio_description/meshes/poignee_collision.stl; visual mesh filename=package://braccio_description/meshes/poignee_visual.stl
- link support_pince: mass None -> 0; geometry collision mesh filename=package://braccio_description/meshes/support_pince_collisio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; visual mesh filename=package://braccio_description/meshes/support_pince_visual.s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
Joints:
- added joint 10f: type fixed, parent part_6_2, child part_1_2, origin xyz=0.000336119 -0.0109949 0.0002 rpy=-3.14159 4.87172e-17 -1.5708, axis 0 0 1, limit effort=1 velocity=20
- added joint 11f: type fixed, parent part_1_2, child part_17, origin xyz=-0.176688 0.011 0.04325 rpy=1.64806e-15 -1.74617e-15 1.5708, axis 0 0 1, limit effort=1 velocity=20
- added joint 13f: type fixed, parent part_6_3, child part_1_3, origin xyz=0.0109949 0.000336119 0.006 rpy=3.14159 1.0011e-14 3.14159, axis 0 0 1, limit effort=1 velocity=20
- added joint 14f: type fixed, parent part_1_3, child part_1_4, origin xyz=-0.1342 -0.0085 0.009 rpy=-3.14159 -2.26416e-31 1.5708, axis 0 0 1, limit effort=1 velocity=20
- added joint 16f: type fixed, parent poignee, child part_11, origin xyz=0.008 0.110686 -0.016 rpy=-1.5708 1.5708 0, axis 0 0 1, limit effort=1 velocity=20
- added joint 18f: type fixed, parent part_2, child support_pince, origin xyz=-2.60209e-18 -8.67362e-19 0.01431 rpy=3.14159 -1.57772e-30 1.5708, axis 0 0 1, limit effort=1 velocity=20
- added joint 19f: type fixed, parent support_pince, child part_11_2, origin xyz=0.00350003 -0.0142499 -0.00999994 rpy=1.5708 -1.5708 0, axis 0 0 1, limit effort=1 velocity=20
- added joint 1f: type fixed, parent base_link, child part_7, origin xyz=-0.011 -0.0478 0.0825 rpy=0 -0 0, axis 0 0 1, limit effort=1 velocity=20
- added joint 21f: type fixed, parent part_2_2, child part_1_5, origin xyz=0 0 -0.0077 rpy=-3.9795e-15 2.22045e-16 -1.5708, axis 0 0 1, limit effort=1 velocity=20
- added joint 22f: type fixed, parent part_1_5, child part_1_6, origin xyz=0.0135856 -0.0828639 0.0525 rpy=-3.14159 3.27525e-30 6.31089e-30, axis 0 0 1, limit effort=1 velocity=20
- added joint 24f: type fixed, parent part_1_7, child part_1_8, origin xyz=-0.0011547 0.002 -0.0375 rpy=-3.14159 -1.11022e-16 -3.14159, axis 0 0 1, limit effort=1 velocity=20
- added joint 25f: type fixed, parent part_1_8, child part_1_9, origin xyz=-0.0111547 -0.002 0.0025 rpy=-9.18292e-15 2.22045e-16 -5.68108e-16, axis 0 0 1, limit effort=1 velocity=20
- added joint 26f: type fixed, parent part_1_7, child part_1_10, origin xyz=6.93889e-18 -2.22045e-16 0.039 rpy=-3.67723e-17 1.72085e-15 -3.14159, axis 0 0 1, limit effort=1 velocity=20
- added joint 3f: type fixed, parent part_6, child part_4, origin xyz=-6.09235e-15 6.45317e-15 -0.0043 rpy=3.14159 1.24298e-32 -5.55112e-17, axis 0 0 1, limit effort=1 velocity=20
- added joint 4f: type fixed, parent part_5, child part_6, origin xyz=-0.000120642 -0.00012451 0.002 rpy=3.14159 7.76538e-31 1.14427e-34, axis 0 0 1, limit effort=1 velocity=20
- added joint 5f: type fixed, parent part_6, child part_1, origin xyz=-6.08888e-15 6.45493e-15 -0.0078 rpy=3.14159 -3.16787e-30 3.14159, axis 0 0 1, limit effort=1 velocity=20
- added joint 6f: type fixed, parent part_1, child part_7_2, origin xyz=0.011 0.01725 0.0203 rpy=-1.5708 7.88861e-31 6.05033e-40, axis 0 0 1, limit effort=1 velocity=20
- added joint 8f: type fixed, parent part_5_2, child part_4_2, origin xyz=1.11131e-18 2.77556e-17 0.0013 rpy=3.14159 -1.23886e-14 -3.14159, axis 0 0 1, limit effort=1 velocity=20
- added joint 9f: type fixed, parent part_4_2, child part_6_2, origin xyz=-8.72783e-18 2.77556e-17 -0.0048 rpy=-3.14159 -1.46256e-30 -5.55112e-17, axis 0 0 1, limit effort=1 velocity=20
- added joint base: type revolute, parent part_7, child part_5, origin xyz=0.011 0.0478 0.004 rpy=1.63909e-22 3.23741e-22 1.5708, axis 0 0 1, limit lower=-4.71239 upper=4.71239 effort=1 velocity=20
- added joint coude: type revolute, parent part_17, child part_6_3, origin xyz=-0.0109994 0.0453 -0.0362 rpy=-3.14159 -1.40621e-15 1.5708, axis 0 0 1, limit lower=-2.0944 upper=2.0944 effort=1 velocity=20
- added joint epaule: type revolute, parent part_7_2, child part_5_2, origin xyz=-0.011 -0.0478 -0.038 rpy=-3.14159 -1.84536e-15 -3.14159, axis 0 0 1, limit lower=-2.0944 upper=2.0944 effort=1 velocity=20
- added joint pince_lib: type revolute, parent support_pince, child part_1_7, origin xyz=0.024 -0.000549949 -0.0234999 rpy=1.5708 -6.66587e-29 -2.94781e-15, axis 0 0 1, limit lower=0 upper=1.5708 effort=1 velocity=20
- added joint pince_mot: type revolute, parent part_11_2, child part_2_2, origin xyz=-0.0135 0.0225 -0.0026 rpy=3.14159 4.31256e-15 5.73896e-29, axis 0 0 1, limit lower=0 upper=1.5708 effort=1 velocity=20
- added joint poignet_incl: type revolute, parent part_1_4, child poignee, origin xyz=0.0080763 -0.0358 0.01475 rpy=-3.8477e-15 1.20224e-15 -3.14159, axis 0 0 1, limit lower=-1.74533 upper=1.74533 effort=1 velocity=20
- added joint poignet_rot: type revolute, parent part_11, child part_2, origin xyz=0.0135 0.0145 -0.0026 rpy=-2.22045e-16 -2.22045e-16 -1.64305e-14, axis 0 0 1, limit lower=-3.14159 upper=3.14159 effort=1 velocity=20

Commit message: rename gripper stl files

File: catkin_ws/src/braccio_description/urdf/robot.urdf (robot description, URDF)
Before this commit: robot onshape, 27 links, 26 joints
Links:
- removed link part_1_10
- removed link part_1_5
- removed link part_1_6
- removed link part_1_7
- removed link part_1_8
- removed link part_1_9
- added link pince, mass 0; collision mesh filename=package://braccio_description/meshes/pince_collision.stl; visual mesh filename=package://braccio_description/meshes/pince_visual.stl
- added link pince_2, mass 0; collision mesh filename=package://braccio_description/meshes/pince_2_collision.stl; visual mesh filename=package://braccio_description/meshes/pince_2_visual.stl
- added link pince_3, mass 0; collision mesh filename=package://braccio_description/meshes/pince_3_collision.stl; visual mesh filename=package://braccio_description/meshes/pince_3_visual.stl
- added link pince_4, mass 0; collision mesh filename=package://braccio_description/meshes/pince_4_collision.stl; visual mesh filename=package://braccio_description/meshes/pince_4_visual.stl
- added link pince_5, mass 0; collision mesh filename=package://braccio_description/meshes/pince_5_collision.stl; visual mesh filename=package://braccio_description/meshes/pince_5_visual.stl
- added link pince_6, mass 0.0598161; collision mesh filename=package://braccio_description/meshes/pince_6_collision.stl; visual mesh filename=package://braccio_description/meshes/pince_6_visual.stl
Joints:
- joint 21f: child part_1_5 -> pince
- joint 22f: child part_1_6 -> pince_2; parent part_1_5 -> pince
- joint 24f: child part_1_8 -> pince_4; parent part_1_7 -> pince_3
- joint 25f: child part_1_9 -> pince_5; parent part_1_8 -> pince_4
- joint 26f: child part_1_10 -> pince_6; parent part_1_7 -> pince_3
- joint pince_lib: child part_1_7 -> pince_3

Commit message: adding braccio_moveit_config package

File: catkin_ws/src/braccio_description/urdf/robot.urdf (robot description, URDF)
Before this commit: robot onshape, 27 links, 26 joints
Links:
- added link socle, mass 0; collision mesh filename=package://braccio_description/meshes/socle_collision.stl; visual mesh filename=package://braccio_description/meshes/socle_visual.stl
Joints:
- added joint 0f: type fixed, parent base_link, child socle, origin xyz=0.0490748 0.0849519 -0.0095 rpy=-3.14159 -2.52904e-15 2.28411e-15, axis 0 0 1, limit effort=1 velocity=20
- joint 1f: origin xyz=-0.011 -0.0478 0.0825 rpy=0 -0 0 -> xyz=-0.0490748 0.0612586 -0.09 rpy=3.14159 1.22465e-16 -3.14159; parent base_link -> socle
- joint 3f: origin xyz=-6.09235e-15 6.45317e-15 -0.0043 rpy=3.14159 1.24298e-32 -5.55112e-17 -> xyz=-6.08714e-15 6.45312e-15 -0.0043 rpy=3.14159 1.24299e-32 -5.55112e-17
- joint 4f: origin xyz=-0.000120642 -0.00012451 0.002 rpy=3.14159 7.76538e-31 1.14427e-34 -> xyz=-0.000120642 -0.00012451 0.002 rpy=3.14159 7.76538e-31 -1.18346e-30
- joint 5f: origin xyz=-6.08888e-15 6.45493e-15 -0.0078 rpy=3.14159 -3.16787e-30 3.14159 -> xyz=-6.08714e-15 6.45249e-15 -0.0098 rpy=-3.14159 4.11812e-22 3.14159
- joint 6f: origin xyz=0.011 0.01725 0.0203 rpy=-1.5708 7.88861e-31 6.05033e-40 -> xyz=0.011 0.01725 0.0203 rpy=-1.5708 4.11812e-22 5.55112e-17
- joint 8f: origin xyz=1.11131e-18 2.77556e-17 0.0013 rpy=3.14159 -1.23886e-14 -3.14159 -> xyz=-2.43945e-18 0 0.0013 rpy=3.14159 -1.23886e-14 -3.14159
- joint 9f: origin xyz=-8.72783e-18 2.77556e-17 -0.0048 rpy=-3.14159 -1.46256e-30 -5.55112e-17 -> xyz=3.38813e-19 0 -0.0048 rpy=-3.14159 -8.8436e-31 -5.55112e-17
- joint base: origin xyz=0.011 0.0478 0.004 rpy=1.63909e-22 3.23741e-22 1.5708 -> xyz=-2.68787e-12 0.0236933 0.004 rpy=3.27819e-22 6.47483e-22 -1.5708
- joint coude: origin xyz=-0.0109994 0.0453 -0.0362 rpy=-3.14159 -1.40621e-15 1.5708 -> xyz=-0.0109994 0.0453 -0.0362 rpy=3.14159 -2.81242e-15 1.5708
- joint epaule: origin xyz=-0.011 -0.0478 -0.038 rpy=-3.14159 -1.84536e-15 -3.14159 -> xyz=-0.011 -0.0478 -0.038 rpy=-3.14159 -3.90704e-15 -3.14159
