Commit message: add collisions to the robot

File: catkin_ws/src/braccio_description/urdf/robot.urdf (robot description, URDF)
Before this commit: robot onshape, 28 links, 27 joints
Links:
- removed link part_1
- removed link part_11
- removed link part_11_2
- removed link part_17
- removed link part_1_2
- removed link part_1_3
- removed link part_1_4
- removed link part_2
- removed link part_2_2
- removed link part_4
- removed link part_4_2
- removed link part_5
- removed link part_5_2
- removed link part_6
- removed link part_6_2
- removed link part_6_3
- removed link part_7
- removed link part_7_2
- removed link pince
- removed link pince_2
- removed link pince_3
- removed link pince_4
- removed link pince_5
- removed link pince_6
- removed link poignee
- added link avant_bras, mass 0; collision box size=0.038 0.14 0.045; collision box size=0.0646 0.093 0.045
- added link bras, mass 0; collision box size=0.0409 0.175 0.045; collision box size=0.0681 0.094 0.045
- added link moteur_bas, mass 0; visual mesh filename=package://braccio_description/meshes/moteur_bas.stl
- added link moteur_bas_2, mass 0; visual mesh filename=package://braccio_description/meshes/moteur_bas.stl
- added link moteur_bas_c1, mass 0; visual mesh filename=package://braccio_description/meshes/moteur_bas_c1.stl
- added link moteur_bas_c1_2, mass 0; visual mesh filename=package://braccio_description/meshes/moteur_bas_c1.stl
- added link moteur_bas_c1_3, mass 0; visual mesh filename=package://braccio_description/meshes/moteur_bas_c1.stl
- added link moteur_bas_c2, mass 0; visual mesh filename=package://braccio_description/meshes/moteur_bas_c2.stl
- added link moteur_bas_c2_2, mass 0; visual mesh filename=package://braccio_description/meshes/moteur_bas_c2.stl
- added link moteur_bas_c3, mass 0; visual mesh filename=package://braccio_description/meshes/moteur_bas_c3.stl
- added link moteur_bas_c3_2, mass 0; visual mesh filename=package://braccio_description/meshes/moteur_bas_c3.stl
- added link moteur_coude, mass 0; visual mesh filename=package://braccio_description/meshes/moteur_coude.stl
- added link moteur_haut, mass 0; visual mesh filename=package://braccio_description/meshes/moteur_haut.stl
- added link moteur_haut_2, mass 0; visual mesh filename=package://braccio_description/meshes/moteur_haut.stl
- added link moteur_poignet_incl, mass 0; visual mesh filename=package://braccio_description/meshes/moteur_poignet_incl.stl
- added link moteur_poignet_rot_c1, mass 0; visual mesh filename=package://braccio_description/meshes/moteur_poignet_rot_c1.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
- added link moteur_poignet_rot_c1_2, mass 0; visual mesh filename=package://braccio_description/meshes/moteur_poignet_rot_c1.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
- added link pince_lib_1, mass 0.0598161; collision box size=0.003 0.084 0.015; collision box size=0.019 0.098 0.061
- added link pince_lib_2, mass 0; visual mesh filename=package://braccio_description/meshes/pince_lib_2.stl
- added link pince_lib_3, mass 0; visual mesh filename=package://braccio_description/meshes/pince_lib_3.stl
- added link pince_lib_4, mass 0; visual mesh filename=package://braccio_description/meshes/pince_lib_4.stl
- added link pince_mot_1, mass 0; collision box size=0.003 0.084 0.015; collision box size=0.019 0.098 0.06
- added link pince_mot_2, mass 0; visual mesh filename=package://braccio_description/meshes/pince_mot_2.stl
- added link poignet, mass 0; collision box size=0.036 0.049 0.06; collision box size=0.043 0.045 0.0405
- added link support_moteur_epaule, mass 0; collision box size=0.0424 0.048 0.09; visual mesh filename=package://braccio_description/meshes/support_moteur_epaule.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
- link base_link: geometry collision box size=0.119 0.19 0.055; collision box size=0.46 0.38 0.13
- link socle: geometry collision box size=0.116 0.097 0.2; collision box size=0.116 0.097 0.2
- link support_pince: geometry collision box size=0.0665 0.0527 0.043; collision cylinder length=0.01 radius=0.016
Joints:
- joint 0f: origin xyz=0.0490748 0.0849519 -0.0095 rpy=-3.14159 -2.52904e-15 2.28411e-15 -> xyz=0.0582138 0.0688761 -0.0341279 rpy=-3.14159 -2.52904e-15 2.28411e-15
- joint 10f: child part_1_2 -> bras; parent part_6_2 -> moteur_bas_c1_2
- joint 11f: child part_17 -> moteur_coude; parent part_1_2 -> bras
- joint 13f: child part_1_3 -> avant_bras; origin xyz=0.0109949 0.000336119 0.006 rpy=3.14159 1.0011e-14 3.14159 -> xyz=0.0109949 0.000336119 0.006 rpy=3.14159 1.0011e-14 -3.14159; parent part_6_3 -> moteur_bas_c1_3
- joint 14f: child part_1_4 -> moteur_poignet_incl; parent part_1_3 -> avant_bras
- joint 16f: child part_11 -> moteur_haut; parent poignee -> poignet
- joint 18f: origin xyz=-2.60209e-18 -8.67362e-19 0.01431 rpy=3.14159 -1.57772e-30 1.5708 -> xyz=-3.46945e-18 3.46945e-18 0.01431 rpy=3.14159 -1.57772e-30 1.5708; parent part_2 -> moteur_poignet_rot_c1
- joint 19f: child part_11_2 -> moteur_haut_2
- joint 1f: child part_7 -> moteur_bas
- joint 21f: child pince -> pince_mot_1; parent part_2_2 -> moteur_poignet_rot_c1_2
- joint 22f: child pince_2 -> pince_mot_2; parent pince -> pince_mot_1
- joint 24f: child pince_4 -> pince_lib_4; parent pince_3 -> pince_lib_3
- joint 25f: child pince_5 -> pince_lib_2; parent pince_4 -> pince_lib_4
- joint 26f: child pince_6 -> pince_lib_1; origin xyz=6.93889e-18 -2.22045e-16 0.039 rpy=-3.67723e-17 1.72085e-15 -3.14159 -> xyz=0 0 0.039 rpy=-3.67723e-17 1.72085e-15 -3.14159; parent pince_3 -> pince_lib_3
- joint 3f: child part_4 -> moteur_bas_c3; origin xyz=-6.08714e-15 6.45312e-15 -0.0043 rpy=3.14159 1.24299e-32 -5.55112e-17 -> xyz=-6.08888e-15 6.45317e-15 -0.0043 rpy=3.14159 1.24299e-32 -5.55112e-17; parent part_6 -> moteur_bas_c1
- joint 4f: child part_6 -> moteur_bas_c1; parent part_5 -> moteur_bas_c2
- joint 5f: child part_1 -> support_moteur_epaule; origin xyz=-6.08714e-15 6.45249e-15 -0.0098 rpy=-3.14159 4.11812e-22 3.14159 -> xyz=-6.08888e-15 6.45317e-15 -0.0098 rpy=-3.14159 4.11812e-22 3.14159; parent part_6 -> moteur_bas_c1
- joint 6f: child part_7_2 -> moteur_bas_2; parent part_1 -> support_moteur_epaule
- joint 8f: child part_4_2 -> moteur_bas_c3_2; origin xyz=-2.43945e-18 0 0.0013 rpy=3.14159 -1.23886e-14 -3.14159 -> xyz=3.46945e-18 0 0.0013 rpy=3.14159 -1.23886e-14 -3.14159; parent part_5_2 -> moteur_bas_c2_2
- joint 9f: child part_6_2 -> moteur_bas_c1_2; origin xyz=3.38813e-19 0 -0.0048 rpy=-3.14159 -8.8436e-31 -5.55112e-17 -> xyz=-3.46945e-18 0 -0.0048 rpy=-3.14159 -8.8436e-31 -5.55112e-17; parent part_4_2 -> moteur_bas_c3_2
- joint base: child part_5 -> moteur_bas_c2; parent part_7 -> moteur_bas
- joint coude: child part_6_3 -> moteur_bas_c1_3; parent part_17 -> moteur_coude
- joint epaule: child part_5_2 -> moteur_bas_c2_2; parent part_7_2 -> moteur_bas_2
- joint pince_lib: child pince_3 -> pince_lib_3
- joint pince_mot: child part_2_2 -> moteur_poignet_rot_c1_2; parent part_11_2 -> moteur_haut_2
- joint poignet_incl: child poignee -> poignet; parent part_1_4 -> moteur_poignet_incl
- joint poignet_rot: child part_2 -> moteur_poignet_rot_c1; parent part_11 -> moteur_haut
